Commit message: successful launch but solo12 not visible

File: gazebo_ros2_control_demos/urdf/solo12.urdf (robot description, URDF)
Before this commit: robot solo, 17 links, 16 joints
Links:
- added link dummy
Joints:
- added joint dummy_joint: type fixed, parent dummy, child base_link

File: ros2_control_demos/ros2_control_demo_description/diffbot_description/gazebo/diffbot.gazebo.xacro (robot description, xacro)
@@ -6,4 +6,10 @@
 <robot xmlns:xacro="http://ros.org/wiki/xacro">
   <xacro:macro name="diffbot_gazebo" params="prefix">
+    <!-- gazebo_ros2_control-->
+    <gazebo>
+      <plugin filename="libgazebo_ros2_control.so" name="gazebo_ros2_control">
+        <parameters>$(find ros2_control_demo_bringup)/config/diffbot_controllers.yaml</parameters>
+      </plugin>
+    </gazebo>
     <!-- Link1 -->
     <gazebo reference="${prefix}base_link">

File: ros2_control_demos/ros2_control_demo_description/rrbot_description/gazebo/rrbot.gazebo.xacro (robot description, xacro)
@@ -9,5 +9,5 @@
     <gazebo>
       <plugin name="gazebo_ros2_control" filename="libgazebo_ros2_control.so">
-        <parameters>$(find ros2_control_demo_bringup)/config/rrbot_gazebo_forward_controller_position.yaml</parameters>
+        <parameters>$(find ros2_control_demo_bringup)/config/rrbot_controllers.yaml</parameters>
       </plugin>
     </gazebo>

File: ros2_control_demos/ros2_control_demo_description/rrbot_description/ros2_control/rrbot.ros2_control.xacro (robot description, xacro)
@@ -3,9 +3,12 @@
   <xacro:macro name="rrbot_ros2_control" params="name prefix">
     <ros2_control name="${name}" type="system">
-      <hardware>
+      <!-- <hardware>
         <plugin>ros2_control_demo_hardware/RRBotSystemPositionOnlyHardware</plugin>
         <param name="example_param_hw_start_duration_sec">0</param>
         <param name="example_param_hw_stop_duration_sec">3.0</param>
         <param name="example_param_hw_slowdown">100</param>
+      </hardware> -->
+      <hardware>
+        <plugin>gazebo_ros2_control/GazeboSystem</plugin>
       </hardware>
       <joint name="${prefix}joint1">

File: ros2_control_demos/ros2_control_demo_description/rrbot_description/urdf/rrbot.urdf.xacro (robot description, xacro)
@@ -13,5 +13,4 @@
   <!-- Import RRBot ros2_control description -->
   <xacro:include filename="$(find rrbot_description)/ros2_control/rrbot.ros2_control.xacro" />
-  <!-- Import RRBot Gazebo Model-->
   <xacro:include filename="$(find rrbot_description)/gazebo/rrbot.gazebo.xacro" />
   <!-- Used for fixing robot -->
