Commit message: added dummy link, working position controller

File: ros2_control_solo/ros2_description_bolt/ros2_control/system_solo.ros2_control.xacro (robot description, xacro)
@@ -14,8 +14,14 @@
           <param name="max">1</param>
         </command_interface>
-        <state_interface name="position">
-        <param name="initial_value">1.0</param>
-      </state_interface>
-        <state_interface name="velocity"/>
+        <command_interface name="velocity">
+          <param name="min">-1</param>
+          <param name="max">1</param>
+        </command_interface>
+        <state_interface name="position">
+          <param name="initial_value">0.0</param>
+        </state_interface>
+        <state_interface name="velocity">
+          <param name="initial_value">0.0</param>
+        </state_interface>
         <state_interface name="effort"/>
       </joint>
@@ -25,6 +31,14 @@
           <param name="max">1</param>
         </command_interface>
-        <state_interface name="position"/>
-        <state_interface name="velocity"/>
+        <command_interface name="velocity">
+          <param name="min">-1</param>
+          <param name="max">1</param>
+        </command_interface>
+        <state_interface name="position">
+          <param name="initial_value">0.0</param>
+        </state_interface>
+        <state_interface name="velocity">
+          <param name="initial_value">0.0</param>
+        </state_interface>
         <state_interface name="effort"/>
       </joint>
@@ -34,6 +48,14 @@
           <param name="max">1</param>
         </command_interface>
-        <state_interface name="position"/>
-        <state_interface name="velocity"/>
+        <command_interface name="velocity">
+          <param name="min">-1</param>
+          <param name="max">1</param>
+        </command_interface>
+        <state_interface name="position">
+          <param name="initial_value">0.0</param>
+        </state_interface>
+        <state_interface name="velocity">
+          <param name="initial_value">0.0</param>
+        </state_interface>
         <state_interface name="effort"/>
       </joint>
@@ -43,6 +65,14 @@
           <param name="max">1</param>
         </command_interface>
-        <state_interface name="position"/>
-        <state_interface name="velocity"/>
+        <command_interface name="velocity">
+          <param name="min">-1</param>
+          <param name="max">1</param>
+        </command_interface>
+        <state_interface name="position">
+          <param name="initial_value">0.0</param>
+        </state_interface>
+        <state_interface name="velocity">
+          <param name="initial_value">0.0</param>
+        </state_interface>
         <state_interface name="effort"/>
       </joint>
@@ -52,6 +82,14 @@
           <param name="max">1</param>
         </command_interface>
-        <state_interface name="position"/>
-        <state_interface name="velocity"/>
+        <command_interface name="velocity">
+          <param name="min">-1</param>
+          <param name="max">1</param>
+        </command_interface>
+        <state_interface name="position">
+          <param name="initial_value">0.0</param>
+        </state_interface>
+        <state_interface name="velocity">
+          <param name="initial_value">0.0</param>
+        </state_interface>
         <state_interface name="effort"/>
       </joint>
@@ -61,6 +99,14 @@
           <param name="max">1</param>
         </command_interface>
-        <state_interface name="position"/>
-        <state_interface name="velocity"/>
+        <command_interface name="velocity">
+          <param name="min">-1</param>
+          <param name="max">1</param>
+        </command_interface>
+        <state_interface name="position">
+          <param name="initial_value">0.0</param>
+        </state_interface>
+        <state_interface name="velocity">
+          <param name="initial_value">0.0</param>
+        </state_interface>
         <state_interface name="effort"/>
       </joint>
@@ -70,6 +116,14 @@
           <param name="max">1</param>
         </command_interface>
-        <state_interface name="position"/>
-        <state_interface name="velocity"/>
+        <command_interface name="velocity">
+          <param name="min">-1</param>
+          <param name="max">1</param>
+        </command_interface>
+        <state_interface name="position">
+          <param name="initial_value">0.0</param>
+        </state_interface>
+        <state_interface name="velocity">
+          <param name="initial_value">0.0</param>
+        </state_interface>
         <state_interface name="effort"/>
       </joint>
@@ -79,6 +133,14 @@
           <param name="max">1</param>
         </command_interface>
-        <state_interface name="position"/>
-        <state_interface name="velocity"/>
+        <command_interface name="velocity">
+          <param name="min">-1</param>
+          <param name="max">1</param>
+        </command_interface>
+        <state_interface name="position">
+          <param name="initial_value">0.0</param>
+        </state_interface>
+        <state_interface name="velocity">
+          <param name="initial_value">0.0</param>
+        </state_interface>
         <state_interface name="effort"/>
       </joint>
@@ -88,6 +150,14 @@
           <param name="max">1</param>
         </command_interface>
-        <state_interface name="position"/>
-        <state_interface name="velocity"/>
+        <command_interface name="velocity">
+          <param name="min">-1</param>
+          <param name="max">1</param>
+        </command_interface>
+        <state_interface name="position">
+          <param name="initial_value">0.0</param>
+        </state_interface>
+        <state_interface name="velocity">
+          <param name="initial_value">0.0</param>
+        </state_interface>
         <state_interface name="effort"/>
       </joint>
@@ -97,6 +167,14 @@
           <param name="max">1</param>
         </command_interface>
-        <state_interface name="position"/>
-        <state_interface name="velocity"/>
+        <command_interface name="velocity">
+          <param name="min">-1</param>
+          <param name="max">1</param>
+        </command_interface>
+        <state_interface name="position">
+          <param name="initial_value">0.0</param>
+        </state_interface>
+        <state_interface name="velocity">
+          <param name="initial_value">0.0</param>
+        </state_interface>
         <state_interface name="effort"/>
       </joint>
@@ -106,6 +184,14 @@
           <param name="max">1</param>
         </command_interface>
-        <state_interface name="position"/>
-        <state_interface name="velocity"/>
+        <command_interface name="velocity">
+          <param name="min">-1</param>
+          <param name="max">1</param>
+        </command_interface>
+        <state_interface name="position">
+          <param name="initial_value">0.0</param>
+        </state_interface>
+        <state_interface name="velocity">
+          <param name="initial_value">0.0</param>
+        </state_interface>
         <state_interface name="effort"/>
       </joint>
@@ -115,6 +201,14 @@
           <param name="max">1</param>
         </command_interface>
-        <state_interface name="position"/>
-        <state_interface name="velocity"/>
+        <command_interface name="velocity">
+          <param name="min">-1</param>
+          <param name="max">1</param>
+        </command_interface>
+        <state_interface name="position">
+          <param name="initial_value">0.0</param>
+        </state_interface>
+        <state_interface name="velocity">
+          <param name="initial_value">0.0</param>
+        </state_interface>
         <state_interface name="effort"/>
       </joint>

File: ros2_control_solo/ros2_description_bolt/urdf/crane.urdf.xacro (robot description, xacro)
@@ -9,7 +9,29 @@
 <robot xmlns:xacro="http://ros.org/wiki/xacro">
   <xacro:macro name="crane" params="parent">
-    <link name="crane_link">
+    <!-- <link name="crane_link">
       <inertial>
-        <origin xyz="0.0 0.0 0" rpy="0.0 0.0 0.0"/>
+        <origin xyz="0 0 0" />
+        <mass value="1.0" />
+        <inertia  ixx="1.0" ixy="0.0"  ixz="0.0"  iyy="100.0"  iyz="0.0"  izz="1.0" />
+      </inertial>
+      <visual>
+        <origin xyz="0 0 0.25"/>
+        <geometry>
+          <box size="0.1 0.1 0.5" />
+        </geometry>
+      </visual>
+    <collision>
+      <origin xyz="0 0 0.05"/>
+      <geometry>
+        <box size="0.1 0.1 0.5" />
+      </geometry>
+    </collision>
+  </link>
+  <gazebo reference="my_box">
+    <material>Gazebo/Blue</material>
+  </gazebo> -->
+    <!-- <link name="crane_link">
+      <inertial>
+        <origin xyz="0.0 0.0 0.0" rpy="0.0 0.0 0.0"/>
         <mass value="0.0"/>
         <inertia ixx="0.0" ixy="0.0" ixz="0.0"
@@ -18,5 +40,35 @@
       </inertial>
       <visual>
-        <origin xyz="-0.25 0 0.0" rpy="0 0 0" />
+        <origin xyz="0.0 0 0.0" rpy="0 0 0" />
+        <geometry>
+          <box size="0.1 0.1 0.1"/>
+        </geometry>
+        <material name="CraneMaterial" rgba="0.3 0.3 0.3 0.1"/>
+      </visual>
+      <collision>
+        <origin xyz="0 0 0" rpy="0 0 0" />
+        <geometry>
+          <box size="0.1 0.1 0.1"/>
+        </geometry>
+        <material name="CraneMaterial"/>
+      </collision>
+    </link> -->
+    <!-- <joint name="crane_joint" type="fixed">
+      <parent link="crane_link" />
+      <child link="${parent}" />
+      <origin xyz="0.003 0.0 -0.1" rpy="0.0  0.0  0.0"/>
+      <limit lower="0.0" upper="0.0" effort="0.0" velocity="0.0" />
+      <dynamics friction="0.0" damping="0.0"/>
+    </joint> -->
+    <!-- <link name="extend_link">
+      <inertial>
+        <origin xyz="0.0 0.0 0.5" rpy="0.0 0.0 0.0"/>
+        <mass value="0.0"/>
+        <inertia ixx="0.0" ixy="0.0" ixz="0.0"
+                 iyy="0.0" iyz="0.0"
+                 izz="0.0"/>
+      </inertial>
+      <visual>
+        <origin xyz="-0.25 0 0.5" rpy="0 0 0" />
         <geometry>
           <box size="0.5 0.03 0.03"/>
@@ -25,5 +77,5 @@
       </visual>
       <collision>
-        <origin xyz="0 0 0.0" rpy="0 0 0" />
+        <origin xyz="0 0 0.5" rpy="0 0 0" />
         <geometry>
           <box size="0.03 0.03 0.5"/>
@@ -32,16 +84,16 @@
       </collision>
     </link>
-    <joint name="crane_joint" type="fixed">
-      <parent link="crane_link" />
+    <joint name="extend_joint" type="fixed">
+      <parent link="extend_link" />
       <child link="${parent}" />
       <origin xyz="0.003 0.0 -0.1" rpy="0.0  0.0  0.0"/>
       <limit lower="0.0" upper="0.0" effort="0.0" velocity="0.0" />
       <dynamics friction="0.0" damping="0.0"/>
-    </joint>
+    </joint> -->
     <link name="world"/>
     <joint name="fixed" type="fixed">
-      <origin xyz="0.0 0.0 0.2" rpy="0.0  0.0  0.0"/>
+      <origin xyz="0.0 0.0 0.0" rpy="0.0  0.0  0.0"/>
       <parent link="world"/>
-      <child link="crane_link"/>
+      <child link="${parent}"/>
     </joint>
   </xacro:macro>

File: ros2_control_solo/ros2_description_bolt/urdf/solo12_description.xacro (robot description, xacro)
@@ -29,4 +29,7 @@
   </gazebo>
   <!-- Might need to add Gazebo reference later-->
+  <!--Attach Crane-->
+    <xacro:include filename="$(find ros2_description_bolt)/urdf/crane.urdf.xacro" />
+    <xacro:crane parent="base_link" />
   <!-- Add the full robot from urdf-->
   <xacro:solo_full

File: ros2_control_solo/ros2_description_bolt/urdf/solo_xacro/leg.xacro (robot description, xacro)
@@ -121,37 +121,9 @@
         </collision>
         <inertial>
-          <mass value="0.14196048"/>
-          <xacro:if value="${is_front}">
-            <xacro:unless value="${is_right}">
-              <!-- HAA body inertia -->
-              <origin xyz="-0.09407251 -0.00438935 0.00001384" rpy="0 0 0" />
-              <inertia ixx="0.00002802" ixy="0.00003687" ixz="-0.00000009"
-                                        iyy="0.00038264" iyz="0.00000000"
-                                                         izz="0.00038050"/>
-            </xacro:unless>
-            <xacro:if value="${is_right}">
-              <!-- HAA body inertia -->
-              <origin xyz="-0.09407251 0.00438935 -0.00001384" rpy="0 0 0" />
-              <inertia ixx="0.00002802" ixy="-0.00003687" ixz="0.00000009"
-                                        iyy="0.00038264"  iyz="0.00000000"
-                                                          izz="0.00038050"/>
-            </xacro:if>
-          </xacro:if>
-          <xacro:unless value="${is_front}">
-            <xacro:unless value="${is_right}">
-              <!-- HAA body inertia -->
-              <origin xyz="0.09407251 -0.00438935 -0.00001384" rpy="0 0 0" />
-              <inertia ixx="0.00002802" ixy="-0.00003687" ixz="-0.00000009"
-                                        iyy="0.00038264"  iyz="0.00000000"
-                                                          izz="0.00038050"/>
-            </xacro:unless>
-            <xacro:if value="${is_right}">
-              <!-- HAA body inertia -->
-              <origin xyz="0.09407251 0.00438935 0.00001384" rpy="0 0 0" />
-              <inertia ixx="0.00002802" ixy="0.00003687" ixz="0.00000009"
-                                        iyy="0.00038264" iyz="0.00000000"
-                                                         izz="0.00038050"/>
-            </xacro:if>
-          </xacro:unless>
+          <!-- <mass value="0.14196048"/> -->
+          <mass value="0.14853845"/>
+          <!-- HAA body inertia -->
+          <origin rpy="0 0 0" xyz="-0.07870700 0.01 0."/>
+          <inertia ixx="0.00003024" ixy="0.00004671" ixz="0.0" iyy="0.00041193" iyz="0.0" izz="0.00041107"/>
         </inertial>
       </link>
@@ -217,9 +189,12 @@
         <!-- Left upper leg inertia -->
         <inertial>
-        <mass value="0.14737324"/>
+        <origin rpy="0 0 0" xyz="0.00001377 0.01935853 -0.07870700"/>
+        <mass value="0.14853845"/>
+        <inertia ixx="0.00041107" ixy="0.0" ixz="0.0" iyy="0.00041193" iyz="0.00004671" izz="0.00003024"/>
+        <!-- <mass value="0.14737324"/>
         <origin xyz="0.00001530 0.01767640 -0.07838230" rpy="0 0 0" />
         <inertia ixx="0.00041540"  ixy="0.00000000" ixz="0.00000010"
                                    iyy="0.00041637" iyz="-0.00004589"
-                                                    izz="0.00002982"/>
+                                                    izz="0.00002982"/> -->
         </inertial>
       </xacro:unless>
@@ -227,9 +202,12 @@
         <!-- Right upper leg inertia -->
         <inertial>
-        <mass value="0.14737324"/>
-        <origin xyz="-0.00001530 -0.01767640 -0.07838230" rpy="0 0 0" />
-        <inertia ixx="0.00041540"  ixy="0.00000000" ixz="-0.00000010"
-                                   iyy="0.00041637" iyz="0.00004589"
-                                                    izz="0.00002982"/>
+        <origin rpy="0 0 0" xyz="0.00001377 0.01935853 -0.07870700"/>
+        <mass value="0.14853845"/>
+        <inertia ixx="0.00041107" ixy="0.0" ixz="0.0" iyy="0.00041193" iyz="0.00004671" izz="0.00003024"/>
+        <!-- <mass value="0.14737324"/>
+        <origin xyz="0.00001530 0.01767640 -0.07838230" rpy="0 0 0" />
+        <inertia ixx="0.00041540"  ixy="0.00000000" ixz="0.00000010"
+                                   iyy="0.00041637" iyz="-0.00004589"
+                                                    izz="0.00002982"/> -->
         </inertial>
       </xacro:if>
@@ -306,9 +284,12 @@
         <!-- Left lower leg inertia -->
         <inertial>
-        <mass value="0.02318294"/>
+        <origin rpy="0 0 0" xyz="0.0 0.00787644 -0.08928215"/>
+        <mass value="0.03070001"/>
+        <inertia ixx="0.00012024" ixy="0.0" ixz="0.0" iyy="0.00012029" iyz="0.00000305" izz="0.00000216"/>
+        <!-- <mass value="0.02318294"/>
         <origin xyz="0.00000000 0.00776716 -0.07003876" rpy="0 0 0" />
         <inertia ixx="0.00008508" ixy="0.00000000"  ixz="0.00000000"
                                   iyy="0.00008580"  iyz="-0.00000200"
-                                                    izz="0.00000139"/>
+                                                    izz="0.00000139"/> -->
         </inertial>
       </xacro:unless>
@@ -316,9 +297,12 @@
         <!-- Right lower leg inertia -->
         <inertial>
-        <mass value="0.02318294"/>
-        <origin xyz="0.00000000 -0.00776716 -0.07003876" rpy="0 0 0" />
+        <origin rpy="0 0 0" xyz="0.0 0.00787644 -0.08928215"/>
+        <mass value="0.03070001"/>
+        <inertia ixx="0.00012024" ixy="0.0" ixz="0.0" iyy="0.00012029" iyz="0.00000305" izz="0.00000216"/>
+        <!-- <mass value="0.02318294"/>
+        <origin xyz="0.00000000 0.00776716 -0.07003876" rpy="0 0 0" />
         <inertia ixx="0.00008508" ixy="0.00000000"  ixz="0.00000000"
-                                  iyy="0.00008580"  iyz="0.00000200"
-                                                    izz="0.00000139"/>
+                                  iyy="0.00008580"  iyz="-0.00000200"
+                                                    izz="0.00000139"/> -->
         </inertial>
       </xacro:if>
@@ -384,9 +368,12 @@
       <!-- FOOT INERTIAL -->
       <inertial>
-        <origin xyz="0 0 0" rpy="0 0 0" />
+        <!-- <origin xyz="0 0 0" rpy="0 0 0" />
         <mass value="0.0"/>
         <inertia ixx="0.0" ixy="0.0" ixz="0.0"
                            iyy="0.0" iyz="0.0"
-                                     izz="0.0"/>
+                                     izz="0.0"/> -->
+      <origin rpy="0 0 0" xyz="0 0 0.00035767"/>
+      <mass value="0.00693606"/>
+      <inertia ixx="0.00000057" ixy="0.0" ixz="0.0" iyy="0.00000084" iyz="0.0" izz="0.00000053"/>
       </inertial>
     </link> <!-- END FOOT LINK -->

File: ros2_control_solo/ros2_description_bolt/urdf/solo_xacro/solo12.urdf.xacro (robot description, xacro)
@@ -15,10 +15,13 @@
       <inertial>
           <origin xyz="-0.00082966 0.00000105 -0.00060210" rpy="0 0 0" />
-          <mass value="1.25123725"/>
+          <!-- <mass value="1.25123725"/> -->
           <!-- The base is extremely symmetrical. -->
-          <inertia ixx="0.00266220" ixy="-0.00003684" ixz="-0.00001716"
+          <!-- <inertia ixx="0.00266220" ixy="-0.00003684" ixz="-0.00001716"
                                     iyy="0.01388510"  iyz="-0.00000009"
                                                       izz="0.01605370"
-          />
+          /> -->
+          <mass value="1.16115091"/>
+          <!-- The base is extremely symmetrical. -->
+          <inertia ixx="0.00578574" ixy="0.0" ixz="0.0" iyy="0.01938108" iyz="0.0" izz="0.02476124"/>
       </inertial>
       <!-- BASE LINK VISUAL -->
