Commit message: fixed inertia errors

File: ros2_control_solo/ros2_description_bolt/ros2_control/system_solo.ros2_control.xacro (robot description, xacro)
@@ -11,33 +11,41 @@
       <joint name="FL_HAA">
         <command_interface name="position">
-          <param name="min">-1</param>
-          <param name="max">1</param>
-        </command_interface>
-        <command_interface name="velocity">
+          <param name="min">-0.9</param>
+          <param name="max">0.9</param>
+        </command_interface>
+        <command_interface name="velocity">
+          <!-- <param name="min">-1</param>
+          <param name="max">1</param> -->
+        </command_interface>
+        <command_interface name="effort">
+          <param name="min">-1</param>
+          <param name="max">1</param>
+        </command_interface>
+       <state_interface name="position">
+          <!-- <param name="initial_value">0.0</param> -->
+        </state_interface>
+        <state_interface name="velocity">
+          <param name="initial_value">0.0</param>
+        </state_interface>
+        <state_interface name="effort"/>
+      </joint>
+      <joint name="FR_HAA">
+        <command_interface name="position">
+          <param name="min">-0.9</param>
+          <param name="max">0.9</param>
+        </command_interface>
+        <command_interface name="velocity">
+          <!-- <param name="min">-1</param>
+          <param name="max">1</param> -->
+        </command_interface>
+        <command_interface name="effort">
           <param name="min">-1</param>
           <param name="max">1</param>
         </command_interface>
         <state_interface name="position">
-          <param name="initial_value">0.0</param>
-        </state_interface>
-        <state_interface name="velocity">
-          <param name="initial_value">0.0</param>
-        </state_interface>
-        <state_interface name="effort"/>
-      </joint>
-      <joint name="FR_HAA">
-        <command_interface name="position">
-          <param name="min">-1</param>
-          <param name="max">1</param>
-        </command_interface>
-        <command_interface name="velocity">
-          <param name="min">-1</param>
-          <param name="max">1</param>
-        </command_interface>
-        <state_interface name="position">
-          <param name="initial_value">0.0</param>
-        </state_interface>
-        <state_interface name="velocity">
-          <param name="initial_value">0.0</param>
+          <!-- <param name="initial_value">0.0</param> -->
+        </state_interface>
+        <state_interface name="velocity">
+          <!-- <param name="initial_value">0.0</param> -->
         </state_interface>
         <state_interface name="effort"/>
@@ -45,16 +53,20 @@
       <joint name="HL_HAA">
         <command_interface name="position">
-          <param name="min">-1</param>
-          <param name="max">1</param>
-        </command_interface>
-        <command_interface name="velocity">
-          <param name="min">-1</param>
-          <param name="max">1</param>
-        </command_interface>
-        <state_interface name="position">
-          <param name="initial_value">0.0</param>
-        </state_interface>
-        <state_interface name="velocity">
-          <param name="initial_value">0.0</param>
+          <param name="min">-0.9</param>
+          <param name="max">0.9</param>
+        </command_interface>
+        <command_interface name="velocity">
+          <!-- <param name="min">-1</param>
+          <param name="max">1</param> -->
+        </command_interface>
+        <command_interface name="effort">
+          <param name="min">-1</param>
+          <param name="max">1</param>
+        </command_interface>
+       <state_interface name="position">
+          <!-- <param name="initial_value">0.0</param> -->
+        </state_interface>
+        <state_interface name="velocity">
+          <!-- <param name="initial_value">0.0</param> -->
         </state_interface>
         <state_interface name="effort"/>
@@ -62,16 +74,20 @@
       <joint name="HR_HAA">
         <command_interface name="position">
-          <param name="min">-1</param>
-          <param name="max">1</param>
-        </command_interface>
-        <command_interface name="velocity">
-          <param name="min">-1</param>
-          <param name="max">1</param>
-        </command_interface>
-        <state_interface name="position">
-          <param name="initial_value">0.0</param>
-        </state_interface>
-        <state_interface name="velocity">
-          <param name="initial_value">0.0</param>
+          <param name="min">-0.9</param>
+          <param name="max">0.9</param>
+        </command_interface>
+        <command_interface name="velocity">
+          <!-- <param name="min">-1</param>
+          <param name="max">1</param> -->
+        </command_interface>
+        <command_interface name="effort">
+          <param name="min">-1</param>
+          <param name="max">1</param>
+        </command_interface>
+       <state_interface name="position">
+          <!-- <param name="initial_value">0.0</param> -->
+        </state_interface>
+        <state_interface name="velocity">
+          <!-- <param name="initial_value">0.0</param> -->
         </state_interface>
         <state_interface name="effort"/>
@@ -79,16 +95,20 @@
       <joint name="FL_HFE">
         <command_interface name="position">
-          <param name="min">-1</param>
-          <param name="max">1</param>
-        </command_interface>
-        <command_interface name="velocity">
-          <param name="min">-1</param>
-          <param name="max">1</param>
-        </command_interface>
-        <state_interface name="position">
-          <param name="initial_value">0.0</param>
-        </state_interface>
-        <state_interface name="velocity">
-          <param name="initial_value">0.0</param>
+          <param name="min">-0.9</param>
+          <param name="max">0.9</param>
+        </command_interface>
+        <command_interface name="velocity">
+          <!-- <param name="min">-1</param>
+          <param name="max">1</param> -->
+        </command_interface>
+        <command_interface name="effort">
+          <param name="min">-1</param>
+          <param name="max">1</param>
+        </command_interface>
+       <state_interface name="position">
+          <!-- <param name="initial_value">0.0</param> -->
+        </state_interface>
+        <state_interface name="velocity">
+          <!-- <param name="initial_value">0.0</param> -->
         </state_interface>
         <state_interface name="effort"/>
@@ -96,16 +116,20 @@
       <joint name="FR_HFE">
         <command_interface name="position">
-          <param name="min">-1</param>
-          <param name="max">1</param>
-        </command_interface>
-        <command_interface name="velocity">
-          <param name="min">-1</param>
-          <param name="max">1</param>
-        </command_interface>
-        <state_interface name="position">
-          <param name="initial_value">0.0</param>
-        </state_interface>
-        <state_interface name="velocity">
-          <param name="initial_value">0.0</param>
+          <param name="min">-0.9</param>
+          <param name="max">0.9</param>
+        </command_interface>
+        <command_interface name="velocity">
+          <!-- <param name="min">-1</param>
+          <param name="max">1</param> -->
+        </command_interface>
+        <command_interface name="effort">
+          <param name="min">-1</param>
+          <param name="max">1</param>
+        </command_interface>
+       <state_interface name="position">
+          <!-- <param name="initial_value">0.0</param> -->
+        </state_interface>
+        <state_interface name="velocity">
+          <!-- <param name="initial_value">0.0</param> -->
         </state_interface>
         <state_interface name="effort"/>
@@ -113,16 +137,20 @@
       <joint name="HL_HFE">
         <command_interface name="position">
-          <param name="min">-1</param>
-          <param name="max">1</param>
-        </command_interface>
-        <command_interface name="velocity">
-          <param name="min">-1</param>
-          <param name="max">1</param>
-        </command_interface>
-        <state_interface name="position">
-          <param name="initial_value">0.0</param>
-        </state_interface>
-        <state_interface name="velocity">
-          <param name="initial_value">0.0</param>
+          <param name="min">-0.9</param>
+          <param name="max">0.9</param>
+        </command_interface>
+        <command_interface name="velocity">
+          <!-- <param name="min">-1</param>
+          <param name="max">1</param> -->
+        </command_interface>
+        <command_interface name="effort">
+          <param name="min">-1</param>
+          <param name="max">1</param>
+        </command_interface>
+       <state_interface name="position">
+          <!-- <param name="initial_value">0.0</param> -->
+        </state_interface>
+        <state_interface name="velocity">
+          <!-- <param name="initial_value">0.0</param> -->
         </state_interface>
         <state_interface name="effort"/>
@@ -130,16 +158,20 @@
       <joint name="HR_HFE">
         <command_interface name="position">
-          <param name="min">-1</param>
-          <param name="max">1</param>
-        </command_interface>
-        <command_interface name="velocity">
-          <param name="min">-1</param>
-          <param name="max">1</param>
-        </command_interface>
-        <state_interface name="position">
-          <param name="initial_value">0.0</param>
-        </state_interface>
-        <state_interface name="velocity">
-          <param name="initial_value">0.0</param>
+          <param name="min">-0.9</param>
+          <param name="max">0.9</param>
+        </command_interface>
+        <command_interface name="velocity">
+          <!-- <param name="min">-1</param>
+          <param name="max">1</param> -->
+        </command_interface>
+        <command_interface name="effort">
+          <param name="min">-1</param>
+          <param name="max">1</param>
+        </command_interface>
+       <state_interface name="position">
+          <!-- <param name="initial_value">0.0</param> -->
+        </state_interface>
+        <state_interface name="velocity">
+          <!-- <param name="initial_value">0.0</param> -->
         </state_interface>
         <state_interface name="effort"/>
@@ -147,16 +179,20 @@
       <joint name="FL_KFE">
         <command_interface name="position">
-          <param name="min">-1</param>
-          <param name="max">1</param>
-        </command_interface>
-        <command_interface name="velocity">
-          <param name="min">-1</param>
-          <param name="max">1</param>
-        </command_interface>
-        <state_interface name="position">
-          <param name="initial_value">0.0</param>
-        </state_interface>
-        <state_interface name="velocity">
-          <param name="initial_value">0.0</param>
+          <param name="min">-0.9</param>
+          <param name="max">0.9</param>
+        </command_interface>
+        <command_interface name="velocity">
+          <!-- <param name="min">-1</param>
+          <param name="max">1</param> -->
+        </command_interface>
+        <command_interface name="effort">
+          <param name="min">-1</param>
+          <param name="max">1</param>
+        </command_interface>
+       <state_interface name="position">
+          <!-- <param name="initial_value">0.0</param> -->
+        </state_interface>
+        <state_interface name="velocity">
+          <!-- <param name="initial_value">0.0</param> -->
         </state_interface>
         <state_interface name="effort"/>
@@ -164,16 +200,20 @@
       <joint name="FR_KFE">
         <command_interface name="position">
-          <param name="min">-1</param>
-          <param name="max">1</param>
-        </command_interface>
-        <command_interface name="velocity">
-          <param name="min">-1</param>
-          <param name="max">1</param>
-        </command_interface>
-        <state_interface name="position">
-          <param name="initial_value">0.0</param>
-        </state_interface>
-        <state_interface name="velocity">
-          <param name="initial_value">0.0</param>
+          <param name="min">-0.9</param>
+          <param name="max">0.9</param>
+        </command_interface>
+        <command_interface name="velocity">
+          <!-- <param name="min">-1</param>
+          <param name="max">1</param> -->
+        </command_interface>
+        <command_interface name="effort">
+          <param name="min">-1</param>
+          <param name="max">1</param>
+        </command_interface>
+       <state_interface name="position">
+          <!-- <param name="initial_value">0.0</param> -->
+        </state_interface>
+        <state_interface name="velocity">
+          <!-- <param name="initial_value">0.0</param> -->
         </state_interface>
         <state_interface name="effort"/>
@@ -181,16 +221,20 @@
       <joint name="HL_KFE">
         <command_interface name="position">
-          <param name="min">-1</param>
-          <param name="max">1</param>
-        </command_interface>
-        <command_interface name="velocity">
-          <param name="min">-1</param>
-          <param name="max">1</param>
-        </command_interface>
-        <state_interface name="position">
-          <param name="initial_value">0.0</param>
-        </state_interface>
-        <state_interface name="velocity">
-          <param name="initial_value">0.0</param>
+          <param name="min">-0.9</param>
+          <param name="max">0.9</param>
+        </command_interface>
+        <command_interface name="velocity">
+          <!-- <param name="min">-1</param>
+          <param name="max">1</param> -->
+        </command_interface>
+        <command_interface name="effort">
+          <param name="min">-1</param>
+          <param name="max">1</param>
+        </command_interface>
+       <state_interface name="position">
+          <!-- <param name="initial_value">0.0</param> -->
+        </state_interface>
+        <state_interface name="velocity">
+          <!-- <param name="initial_value">0.0</param> -->
         </state_interface>
         <state_interface name="effort"/>
@@ -198,16 +242,20 @@
       <joint name="HR_KFE">
         <command_interface name="position">
-          <param name="min">-1</param>
-          <param name="max">1</param>
-        </command_interface>
-        <command_interface name="velocity">
-          <param name="min">-1</param>
-          <param name="max">1</param>
-        </command_interface>
-        <state_interface name="position">
-          <param name="initial_value">0.0</param>
-        </state_interface>
-        <state_interface name="velocity">
-          <param name="initial_value">0.0</param>
+          <param name="min">-0.9</param>
+          <param name="max">0.9</param>
+        </command_interface>
+        <command_interface name="velocity">
+          <!-- <param name="min">-1</param>
+          <param name="max">1</param> -->
+        </command_interface>
+        <command_interface name="effort">
+          <param name="min">-1</param>
+          <param name="max">1</param>
+        </command_interface>
+       <state_interface name="position">
+          <!-- <param name="initial_value">0.0</param> -->
+        </state_interface>
+        <state_interface name="velocity">
+          <!-- <param name="initial_value">0.0</param> -->
         </state_interface>
         <state_interface name="effort"/>

File: ros2_control_solo/ros2_description_bolt/urdf/solo12_description.xacro (robot description, xacro)
@@ -30,6 +30,6 @@
   <!-- Might need to add Gazebo reference later-->
   <!--Attach Crane-->
-    <xacro:include filename="$(find ros2_description_bolt)/urdf/crane.urdf.xacro" />
-    <xacro:crane parent="base_link" />
+    <!-- <xacro:include filename="$(find ros2_description_bolt)/urdf/crane.urdf.xacro" />
+    <xacro:crane parent="base_link" /> -->
   <!-- Add the full robot from urdf-->
   <xacro:solo_full
