Commit message: fixed inertia errors

File: ros2_control_solo/ros2_description_bolt/urdf/solo_xacro/leg.xacro (robot description, xacro)
@@ -121,9 +121,37 @@
         </collision>
         <inertial>
-          <!-- <mass value="0.14196048"/> -->
-          <mass value="0.14853845"/>
-          <!-- HAA body inertia -->
-          <origin rpy="0 0 0" xyz="-0.07870700 0.01 0."/>
-          <inertia ixx="0.00003024" ixy="0.00004671" ixz="0.0" iyy="0.00041193" iyz="0.0" izz="0.00041107"/>
+          <mass value="0.14196048"/>
+          <xacro:if value="${is_front}">
+            <xacro:unless value="${is_right}">
+              <!-- HAA body inertia -->
+              <origin xyz="-0.09407251 -0.00438935 0.00001384" rpy="0 0 0" />
+              <inertia ixx="0.00002802" ixy="0.00003687" ixz="-0.00000009"
+                                        iyy="0.00038264" iyz="0.00000000"
+                                                         izz="0.00038050"/>
+            </xacro:unless>
+            <xacro:if value="${is_right}">
+              <!-- HAA body inertia -->
+              <origin xyz="-0.09407251 0.00438935 -0.00001384" rpy="0 0 0" />
+              <inertia ixx="0.00002802" ixy="-0.00003687" ixz="0.00000009"
+                                        iyy="0.00038264"  iyz="0.00000000"
+                                                          izz="0.00038050"/>
+            </xacro:if>
+          </xacro:if>
+          <xacro:unless value="${is_front}">
+            <xacro:unless value="${is_right}">
+              <!-- HAA body inertia -->
+              <origin xyz="0.09407251 -0.00438935 -0.00001384" rpy="0 0 0" />
+              <inertia ixx="0.00002802" ixy="-0.00003687" ixz="-0.00000009"
+                                        iyy="0.00038264"  iyz="0.00000000"
+                                                          izz="0.00038050"/>
+            </xacro:unless>
+            <xacro:if value="${is_right}">
+              <!-- HAA body inertia -->
+              <origin xyz="0.09407251 0.00438935 0.00001384" rpy="0 0 0" />
+              <inertia ixx="0.00002802" ixy="0.00003687" ixz="0.00000009"
+                                        iyy="0.00038264" iyz="0.00000000"
+                                                         izz="0.00038050"/>
+            </xacro:if>
+          </xacro:unless>
         </inertial>
       </link>
@@ -189,12 +217,12 @@
         <!-- Left upper leg inertia -->
         <inertial>
-        <origin rpy="0 0 0" xyz="0.00001377 0.01935853 -0.07870700"/>
-        <mass value="0.14853845"/>
-        <inertia ixx="0.00041107" ixy="0.0" ixz="0.0" iyy="0.00041193" iyz="0.00004671" izz="0.00003024"/>
-        <!-- <mass value="0.14737324"/>
+        <!-- <origin rpy="0 0 0" xyz="0.00001377 0.01935853 -0.07870700"/> -->
+        <!-- <mass value="0.14853845"/> -->
+        <!-- <inertia ixx="0.00041107" ixy="0.0" ixz="0.0" iyy="0.00041193" iyz="0.00004671" izz="0.00003024"/> -->
+        <mass value="0.14737324"/>
         <origin xyz="0.00001530 0.01767640 -0.07838230" rpy="0 0 0" />
         <inertia ixx="0.00041540"  ixy="0.00000000" ixz="0.00000010"
                                    iyy="0.00041637" iyz="-0.00004589"
-                                                    izz="0.00002982"/> -->
+                                                    izz="0.00002982"/>
         </inertial>
       </xacro:unless>
@@ -202,12 +230,12 @@
         <!-- Right upper leg inertia -->
         <inertial>
-        <origin rpy="0 0 0" xyz="0.00001377 0.01935853 -0.07870700"/>
-        <mass value="0.14853845"/>
-        <inertia ixx="0.00041107" ixy="0.0" ixz="0.0" iyy="0.00041193" iyz="0.00004671" izz="0.00003024"/>
-        <!-- <mass value="0.14737324"/>
-        <origin xyz="0.00001530 0.01767640 -0.07838230" rpy="0 0 0" />
-        <inertia ixx="0.00041540"  ixy="0.00000000" ixz="0.00000010"
-                                   iyy="0.00041637" iyz="-0.00004589"
-                                                    izz="0.00002982"/> -->
+        <!-- <origin rpy="0 0 0" xyz="0.00001377 0.01935853 -0.07870700"/> -->
+        <!-- <mass value="0.14853845"/> -->
+        <!-- <inertia ixx="0.00041107" ixy="0.0" ixz="0.0" iyy="0.00041193" iyz="0.00004671" izz="0.00003024"/> -->
+        <mass value="0.14737324"/>
+        <origin xyz="-0.00001530 -0.01767640 -0.07838230" rpy="0 0 0" />
+        <inertia ixx="0.00041540"  ixy="0.00000000" ixz="-0.00000010"
+                                   iyy="0.00041637" iyz="0.00004589"
+                                                    izz="0.00002982"/>
         </inertial>
       </xacro:if>
@@ -284,12 +312,12 @@
         <!-- Left lower leg inertia -->
         <inertial>
-        <origin rpy="0 0 0" xyz="0.0 0.00787644 -0.08928215"/>
-        <mass value="0.03070001"/>
-        <inertia ixx="0.00012024" ixy="0.0" ixz="0.0" iyy="0.00012029" iyz="0.00000305" izz="0.00000216"/>
-        <!-- <mass value="0.02318294"/>
+        <!-- <origin rpy="0 0 0" xyz="0.0 0.00787644 -0.08928215"/> -->
+        <!-- <mass value="0.03070001"/> -->
+        <!-- <inertia ixx="0.00012024" ixy="0.0" ixz="0.0" iyy="0.00012029" iyz="0.00000305" izz="0.00000216"/> -->
+        <mass value="0.02318294"/>
         <origin xyz="0.00000000 0.00776716 -0.07003876" rpy="0 0 0" />
         <inertia ixx="0.00008508" ixy="0.00000000"  ixz="0.00000000"
                                   iyy="0.00008580"  iyz="-0.00000200"
-                                                    izz="0.00000139"/> -->
+                                                    izz="0.00000139"/>
         </inertial>
       </xacro:unless>
@@ -297,12 +325,12 @@
         <!-- Right lower leg inertia -->
         <inertial>
-        <origin rpy="0 0 0" xyz="0.0 0.00787644 -0.08928215"/>
-        <mass value="0.03070001"/>
-        <inertia ixx="0.00012024" ixy="0.0" ixz="0.0" iyy="0.00012029" iyz="0.00000305" izz="0.00000216"/>
-        <!-- <mass value="0.02318294"/>
-        <origin xyz="0.00000000 0.00776716 -0.07003876" rpy="0 0 0" />
+        <!-- <origin rpy="0 0 0" xyz="0.0 0.00787644 -0.08928215"/> -->
+        <!-- <mass value="0.03070001"/> -->
+        <!-- <inertia ixx="0.00012024" ixy="0.0" ixz="0.0" iyy="0.00012029" iyz="0.00000305" izz="0.00000216"/> -->
+        <mass value="0.02318294"/>
+        <origin xyz="0.00000000 -0.00776716 -0.07003876" rpy="0 0 0" />
         <inertia ixx="0.00008508" ixy="0.00000000"  ixz="0.00000000"
-                                  iyy="0.00008580"  iyz="-0.00000200"
-                                                    izz="0.00000139"/> -->
+                                  iyy="0.00008580"  iyz="0.00000200"
+                                                    izz="0.00000139"/>
         </inertial>
       </xacro:if>
@@ -368,12 +396,12 @@
       <!-- FOOT INERTIAL -->
       <inertial>
-        <!-- <origin xyz="0 0 0" rpy="0 0 0" />
+        <origin xyz="0 0 0" rpy="0 0 0" />
         <mass value="0.0"/>
         <inertia ixx="0.0" ixy="0.0" ixz="0.0"
                            iyy="0.0" iyz="0.0"
-                                     izz="0.0"/> -->
-      <origin rpy="0 0 0" xyz="0 0 0.00035767"/>
-      <mass value="0.00693606"/>
-      <inertia ixx="0.00000057" ixy="0.0" ixz="0.0" iyy="0.00000084" iyz="0.0" izz="0.00000053"/>
+                                     izz="0.0"/>
+      <!-- <origin rpy="0 0 0" xyz="0 0 0.00035767"/> -->
+      <!-- <mass value="0.00693606"/> -->
+      <!-- <inertia ixx="0.00000057" ixy="0.0" ixz="0.0" iyy="0.00000084" iyz="0.0" izz="0.00000053"/> -->
       </inertial>
     </link> <!-- END FOOT LINK -->

File: ros2_control_solo/ros2_description_bolt/urdf/solo_xacro/solo12.urdf.xacro (robot description, xacro)
@@ -15,13 +15,13 @@
       <inertial>
           <origin xyz="-0.00082966 0.00000105 -0.00060210" rpy="0 0 0" />
-          <!-- <mass value="1.25123725"/> -->
+          <mass value="1.25123725"/>
           <!-- The base is extremely symmetrical. -->
-          <!-- <inertia ixx="0.00266220" ixy="-0.00003684" ixz="-0.00001716"
+          <inertia ixx="0.00266220" ixy="-0.00003684" ixz="-0.00001716"
                                     iyy="0.01388510"  iyz="-0.00000009"
                                                       izz="0.01605370"
-          /> -->
-          <mass value="1.16115091"/>
+          />
+          <!-- <mass value="1.16115091"/> -->
           <!-- The base is extremely symmetrical. -->
-          <inertia ixx="0.00578574" ixy="0.0" ixz="0.0" iyy="0.01938108" iyz="0.0" izz="0.02476124"/>
+          <!-- <inertia ixx="0.00578574" ixy="0.0" ixz="0.0" iyy="0.01938108" iyz="0.0" izz="0.02476124"/> -->
       </inertial>
       <!-- BASE LINK VISUAL -->

File: ros2_control_solo/ros2_description_bolt/urdf/system_bolt_description.urdf.xacro (robot description, xacro)
@@ -17,5 +17,5 @@
   <xacro:arg name="prefix" default="" />
   <xacro:arg name="use_crane" default="true" />
-  <xacro:arg name="use_sim" default="false" />
+  <xacro:arg name="use_sim" default="true" />
   <xacro:arg name="use_fake_hardware" default="false" />
   <!-- Include the legs -->

Commit message: for_pos_controller

File: ros2_control_solo/ros2_description_bolt/ros2_control/system_solo.ros2_control.xacro (robot description, xacro)
@@ -4,5 +4,5 @@
 <!-- Examples: https://github.com/ros-controls/ros2_control_demos -->
 <robot xmlns:xacro="http://www.ros.org/wiki/xacro">
-  <xacro:macro name="system_solo_ros2_control" params="name prefix use_sim:=^|false use_fake_hardware:=^|true fake_sensor_commands:=^|false slowdown:=2.0 ethernet_port:=^|enp6s0f1 true:=^|true false:=^|false">
+  <xacro:macro name="system_solo_ros2_control" params="name">
     <ros2_control name="${name}" type="system">
       <hardware>
@@ -11,20 +11,10 @@
       <joint name="FL_HAA">
         <command_interface name="position">
-          <param name="min">-0.9</param>
-          <param name="max">0.9</param>
-        </command_interface>
-        <command_interface name="velocity">
-          <!-- <param name="min">-1</param>
-          <param name="max">1</param> -->
-        </command_interface>
-        <command_interface name="effort">
-          <param name="min">-1</param>
-          <param name="max">1</param>
+          <param name="min">-3.14</param>
+          <param name="max">3.14</param>
         </command_interface>
        <state_interface name="position">
-          <!-- <param name="initial_value">0.0</param> -->
         </state_interface>
         <state_interface name="velocity">
-          <param name="initial_value">0.0</param>
         </state_interface>
         <state_interface name="effort"/>
@@ -32,20 +22,10 @@
       <joint name="FR_HAA">
         <command_interface name="position">
-          <param name="min">-0.9</param>
-          <param name="max">0.9</param>
-        </command_interface>
-        <command_interface name="velocity">
-          <!-- <param name="min">-1</param>
-          <param name="max">1</param> -->
-        </command_interface>
-        <command_interface name="effort">
-          <param name="min">-1</param>
-          <param name="max">1</param>
+          <param name="min">-3.14</param>
+          <param name="max">3.14</param>
         </command_interface>
         <state_interface name="position">
-          <!-- <param name="initial_value">0.0</param> -->
         </state_interface>
         <state_interface name="velocity">
-          <!-- <param name="initial_value">0.0</param> -->
         </state_interface>
         <state_interface name="effort"/>
@@ -53,20 +33,10 @@
       <joint name="HL_HAA">
         <command_interface name="position">
-          <param name="min">-0.9</param>
-          <param name="max">0.9</param>
-        </command_interface>
-        <command_interface name="velocity">
-          <!-- <param name="min">-1</param>
-          <param name="max">1</param> -->
-        </command_interface>
-        <command_interface name="effort">
-          <param name="min">-1</param>
-          <param name="max">1</param>
+          <param name="min">-3.14</param>
+          <param name="max">3.14</param>
         </command_interface>
        <state_interface name="position">
-          <!-- <param name="initial_value">0.0</param> -->
         </state_interface>
         <state_interface name="velocity">
-          <!-- <param name="initial_value">0.0</param> -->
         </state_interface>
         <state_interface name="effort"/>
@@ -74,20 +44,10 @@
       <joint name="HR_HAA">
         <command_interface name="position">
-          <param name="min">-0.9</param>
-          <param name="max">0.9</param>
-        </command_interface>
-        <command_interface name="velocity">
-          <!-- <param name="min">-1</param>
-          <param name="max">1</param> -->
-        </command_interface>
-        <command_interface name="effort">
-          <param name="min">-1</param>
-          <param name="max">1</param>
+          <param name="min">-3.14</param>
+          <param name="max">3.14</param>
         </command_interface>
        <state_interface name="position">
-          <!-- <param name="initial_value">0.0</param> -->
         </state_interface>
         <state_interface name="velocity">
-          <!-- <param name="initial_value">0.0</param> -->
         </state_interface>
         <state_interface name="effort"/>
@@ -95,20 +55,11 @@
       <joint name="FL_HFE">
         <command_interface name="position">
-          <param name="min">-0.9</param>
-          <param name="max">0.9</param>
-        </command_interface>
-        <command_interface name="velocity">
-          <!-- <param name="min">-1</param>
-          <param name="max">1</param> -->
-        </command_interface>
-        <command_interface name="effort">
-          <param name="min">-1</param>
-          <param name="max">1</param>
+          <param name="min">-3.14</param>
+          <param name="max">3.14</param>
         </command_interface>
        <state_interface name="position">
-          <!-- <param name="initial_value">0.0</param> -->
+          <param name="initial_value">1.57</param>
         </state_interface>
         <state_interface name="velocity">
-          <!-- <param name="initial_value">0.0</param> -->
         </state_interface>
         <state_interface name="effort"/>
@@ -116,20 +67,11 @@
       <joint name="FR_HFE">
         <command_interface name="position">
-          <param name="min">-0.9</param>
-          <param name="max">0.9</param>
-        </command_interface>
-        <command_interface name="velocity">
-          <!-- <param name="min">-1</param>
-          <param name="max">1</param> -->
-        </command_interface>
-        <command_interface name="effort">
-          <param name="min">-1</param>
-          <param name="max">1</param>
+          <param name="min">-3.14</param>
+          <param name="max">3.14</param>
         </command_interface>
        <state_interface name="position">
-          <!-- <param name="initial_value">0.0</param> -->
+          <param name="initial_value">1.57</param>
         </state_interface>
         <state_interface name="velocity">
-          <!-- <param name="initial_value">0.0</param> -->
         </state_interface>
         <state_interface name="effort"/>
@@ -137,20 +79,11 @@
       <joint name="HL_HFE">
         <command_interface name="position">
-          <param name="min">-0.9</param>
-          <param name="max">0.9</param>
-        </command_interface>
-        <command_interface name="velocity">
-          <!-- <param name="min">-1</param>
-          <param name="max">1</param> -->
-        </command_interface>
-        <command_interface name="effort">
-          <param name="min">-1</param>
-          <param name="max">1</param>
+          <param name="min">-3.14</param>
+          <param name="max">3.14</param>
         </command_interface>
        <state_interface name="position">
-          <!-- <param name="initial_value">0.0</param> -->
+          <param name="initial_value">-1.57</param>
         </state_interface>
         <state_interface name="velocity">
-          <!-- <param name="initial_value">0.0</param> -->
         </state_interface>
         <state_interface name="effort"/>
@@ -158,20 +91,11 @@
       <joint name="HR_HFE">
         <command_interface name="position">
-          <param name="min">-0.9</param>
-          <param name="max">0.9</param>
-        </command_interface>
-        <command_interface name="velocity">
-          <!-- <param name="min">-1</param>
-          <param name="max">1</param> -->
-        </command_interface>
-        <command_interface name="effort">
-          <param name="min">-1</param>
-          <param name="max">1</param>
+          <param name="min">-3.14</param>
+          <param name="max">3.14</param>
         </command_interface>
        <state_interface name="position">
-          <!-- <param name="initial_value">0.0</param> -->
+          <param name="initial_value">-1.57</param>
         </state_interface>
         <state_interface name="velocity">
-          <!-- <param name="initial_value">0.0</param> -->
         </state_interface>
         <state_interface name="effort"/>
@@ -179,20 +103,11 @@
       <joint name="FL_KFE">
         <command_interface name="position">
-          <param name="min">-0.9</param>
-          <param name="max">0.9</param>
-        </command_interface>
-        <command_interface name="velocity">
-          <!-- <param name="min">-1</param>
-          <param name="max">1</param> -->
-        </command_interface>
-        <command_interface name="effort">
-          <param name="min">-1</param>
-          <param name="max">1</param>
+          <param name="min">-3.14</param>
+          <param name="max">3.14</param>
         </command_interface>
        <state_interface name="position">
-          <!-- <param name="initial_value">0.0</param> -->
+          <param name="initial_value">3.14</param>
         </state_interface>
         <state_interface name="velocity">
-          <!-- <param name="initial_value">0.0</param> -->
         </state_interface>
         <state_interface name="effort"/>
@@ -200,20 +115,11 @@
       <joint name="FR_KFE">
         <command_interface name="position">
-          <param name="min">-0.9</param>
-          <param name="max">0.9</param>
-        </command_interface>
-        <command_interface name="velocity">
-          <!-- <param name="min">-1</param>
-          <param name="max">1</param> -->
-        </command_interface>
-        <command_interface name="effort">
-          <param name="min">-1</param>
-          <param name="max">1</param>
+          <param name="min">-3.14</param>
+          <param name="max">3.14</param>
         </command_interface>
        <state_interface name="position">
-          <!-- <param name="initial_value">0.0</param> -->
+          <param name="initial_value">3.14</param>
         </state_interface>
         <state_interface name="velocity">
-          <!-- <param name="initial_value">0.0</param> -->
         </state_interface>
         <state_interface name="effort"/>
@@ -221,20 +127,11 @@
       <joint name="HL_KFE">
         <command_interface name="position">
-          <param name="min">-0.9</param>
-          <param name="max">0.9</param>
-        </command_interface>
-        <command_interface name="velocity">
-          <!-- <param name="min">-1</param>
-          <param name="max">1</param> -->
-        </command_interface>
-        <command_interface name="effort">
-          <param name="min">-1</param>
-          <param name="max">1</param>
+          <param name="min">-3.14</param>
+          <param name="max">3.14</param>
         </command_interface>
        <state_interface name="position">
-          <!-- <param name="initial_value">0.0</param> -->
+          <param name="initial_value">3.14</param>
         </state_interface>
         <state_interface name="velocity">
-          <!-- <param name="initial_value">0.0</param> -->
         </state_interface>
         <state_interface name="effort"/>
@@ -242,20 +139,11 @@
       <joint name="HR_KFE">
         <command_interface name="position">
-          <param name="min">-0.9</param>
-          <param name="max">0.9</param>
-        </command_interface>
-        <command_interface name="velocity">
-          <!-- <param name="min">-1</param>
-          <param name="max">1</param> -->
-        </command_interface>
-        <command_interface name="effort">
-          <param name="min">-1</param>
-          <param name="max">1</param>
+          <param name="min">-3.14</param>
+          <param name="max">3.14</param>
         </command_interface>
        <state_interface name="position">
-          <!-- <param name="initial_value">0.0</param> -->
+          <param name="initial_value">3.14</param>
         </state_interface>
         <state_interface name="velocity">
-          <!-- <param name="initial_value">0.0</param> -->
         </state_interface>
         <state_interface name="effort"/>

File: ros2_control_solo/ros2_description_bolt/urdf/solo12_description.xacro (robot description, xacro)
@@ -13,8 +13,4 @@
   <xacro:property name="color" value="0.8 0.8 0.8" />
   <xacro:property name="opacity" value="1.0" />
-  <xacro:arg name="prefix" default="" />
-  <xacro:arg name="use_crane" default="true" />
-  <xacro:arg name="use_sim" default="false" />
-  <xacro:arg name="use_fake_hardware" default="false" />
   <!-- Include the urdf -->
   <xacro:include filename="$(find ros2_description_bolt)/urdf/solo_xacro/solo12.urdf.xacro"/>
@@ -39,6 +35,4 @@
       opacity="${opacity}"/>
   <!-- Add the System from ros2_control-->
-  <xacro:system_solo_ros2_control
-    name="SystemRos2Control" prefix="$(arg prefix)" use_fake_hardware="$(arg use_fake_hardware)"
-      use_sim="$(arg use_sim)"/>
+  <xacro:system_solo_ros2_control name="SystemRos2Control"/>
 </robot>

File: ros2_control_solo/ros2_description_bolt/urdf/solo_xacro/solo12.urdf.xacro (robot description, xacro)
@@ -5,8 +5,8 @@
   xmlns:sensor="http://playerstage.sourceforge.net/gazebo/xmlschema/#sensor"
   xmlns:xacro="http://playerstage.sourceforge.net/gazebo/xmlschema/#interface">
-  <!-- <xacro:property name="color_name" value="grey" />
+  <xacro:property name="color_name" value="grey" />
   <xacro:property name="color" value="0.8 0.8 0.8" />
   <xacro:property name="opacity" value="1.0" />
-  <xacro:property name="mesh_ext" value="stl" /> -->
+  <xacro:property name="mesh_ext" value="stl" />
   <xacro:macro name="solo_full" params="mesh_ext color_name color opacity">
     <!-- This file is based on: https://github.com/open-dynamic-robot-initiative/open_robot_actuator_hardware/blob/master/mechanics/quadruped_robot_12dof_v1/README.md#quadruped-robot-12dof-v1 -->
