Commit message: fixed most of the physics, controller not crashing upon spawn

File: ros2_control_solo/ros2_description_bolt/ros2_control/system_solo.ros2_control.xacro (robot description, xacro)
@@ -14,8 +14,6 @@
           <param name="max">3.14</param>
         </command_interface>
-       <state_interface name="position">
-        </state_interface>
-        <state_interface name="velocity">
-        </state_interface>
+       <state_interface name="position"/>
+        <state_interface name="velocity"/>
         <state_interface name="effort"/>
       </joint>
@@ -25,8 +23,6 @@
           <param name="max">3.14</param>
         </command_interface>
-        <state_interface name="position">
-        </state_interface>
-        <state_interface name="velocity">
-        </state_interface>
+        <state_interface name="position"/>
+        <state_interface name="velocity"/>
         <state_interface name="effort"/>
       </joint>
@@ -36,8 +32,6 @@
           <param name="max">3.14</param>
         </command_interface>
-       <state_interface name="position">
-        </state_interface>
-        <state_interface name="velocity">
-        </state_interface>
+       <state_interface name="position"/>
+        <state_interface name="velocity"/>
         <state_interface name="effort"/>
       </joint>
@@ -47,8 +41,6 @@
           <param name="max">3.14</param>
         </command_interface>
-       <state_interface name="position">
-        </state_interface>
-        <state_interface name="velocity">
-        </state_interface>
+       <state_interface name="position"/>
+        <state_interface name="velocity"/>
         <state_interface name="effort"/>
       </joint>
@@ -59,5 +51,5 @@
         </command_interface>
        <state_interface name="position">
-          <param name="initial_value">1.57</param>
+          <!-- <param name="initial_value">1.57</param> -->
         </state_interface>
         <state_interface name="velocity">
@@ -71,5 +63,5 @@
         </command_interface>
        <state_interface name="position">
-          <param name="initial_value">1.57</param>
+          <!-- <param name="initial_value">1.57</param> -->
         </state_interface>
         <state_interface name="velocity">
@@ -83,5 +75,5 @@
         </command_interface>
        <state_interface name="position">
-          <param name="initial_value">-1.57</param>
+          <!-- <param name="initial_value">-1.57</param> -->
         </state_interface>
         <state_interface name="velocity">
@@ -95,5 +87,5 @@
         </command_interface>
        <state_interface name="position">
-          <param name="initial_value">-1.57</param>
+          <!-- <param name="initial_value">-1.57</param> -->
         </state_interface>
         <state_interface name="velocity">
@@ -107,5 +99,5 @@
         </command_interface>
        <state_interface name="position">
-          <param name="initial_value">3.14</param>
+          <!-- <param name="initial_value">3.14</param> -->
         </state_interface>
         <state_interface name="velocity">
@@ -119,5 +111,5 @@
         </command_interface>
        <state_interface name="position">
-          <param name="initial_value">3.14</param>
+          <!-- <param name="initial_value">3.14</param> -->
         </state_interface>
         <state_interface name="velocity">
@@ -131,5 +123,5 @@
         </command_interface>
        <state_interface name="position">
-          <param name="initial_value">3.14</param>
+          <!-- <param name="initial_value">3.14</param> -->
         </state_interface>
         <state_interface name="velocity">
@@ -143,5 +135,5 @@
         </command_interface>
        <state_interface name="position">
-          <param name="initial_value">3.14</param>
+          <!-- <param name="initial_value">3.14</param> -->
         </state_interface>
         <state_interface name="velocity">
