Commit message: fixed most of the physics, controller not crashing upon spawn

File: ros2_control_solo/ros2_description_bolt/urdf/solo_xacro/leg.xacro (robot description, xacro)
@@ -16,9 +16,12 @@
   <xacro:macro name="leg" params="prefix is_front is_right has_side_motion
                                   mesh_ext color_name color opacity">
+  <!-- HAVE SIDE MOTION -->
     <xacro:if value="${has_side_motion}">
+    <!-- HAA JOINT -->
       <joint name="${prefix}_HAA" type="revolute">
         <parent link="base_link"/>
         <child link="${prefix}_SHOULDER"/>
-        <limit effort="1000" lower="-10" upper="10" velocity="1000"/>
+        <!-- <limit effort="1000" lower="-10" upper="10" velocity="1000"/> -->
+        <limit lower="-1.57" upper="1.57" velocity="1" effort="7"/>
         <!-- joints rotates around the x-axis -->
         <axis xyz="1 0 0"/>
@@ -41,8 +44,9 @@
         </xacro:unless>
         <!-- pybullet simulation parameters -->
-        <dynamics damping="0.0" friction="0.0"/>
+        <dynamics friction="10.0"/>
+        <!-- <dynamics damping="0.0" friction="0.0"/> -->
       </joint>
+    <!-- SHOULDER LINK -->
       <link name="${prefix}_SHOULDER">
-        <!-- HAA VISUAL -->
         <visual>
             <xacro:unless value="${is_right}">
@@ -156,8 +160,10 @@
         </inertial>
       </link>
+  <!-- HFE JOINT -->
       <joint name="${prefix}_HFE" type="revolute">
         <parent link="${prefix}_SHOULDER"/>
         <child link="${prefix}_UPPER_LEG"/>
-        <limit effort="1000" lower="-10" upper="10" velocity="1000"/>
+        <!-- <limit effort="1000" lower="-10" upper="10" velocity="1000"/> -->
+        <limit lower="-3.14" upper="3.14" velocity="1" effort="7"/>
         <!-- joints rotates around the y-axis -->
         <axis xyz="0 1 0"/>
@@ -180,7 +186,174 @@
         </xacro:unless>
         <!-- pybullet simulation parameters -->
-        <dynamics damping="0.0" friction="0.0"/>
+        <!-- <dynamics damping="0.0" friction="0.0"/> -->
+        <dynamics friction="10.0"/>
       </joint>
     </xacro:if>
+  <!-- UPPER LEG LINK -->
+    <link name="${prefix}_UPPER_LEG">
+      <!-- UPPER LEG LINK INERTIAL -->
+      <xacro:unless value="${is_right}">
+        <!-- Left upper leg inertia -->
+        <inertial>
+          <mass value="0.14737324"/>
+          <origin xyz="0.00001530 0.01767640 -0.07838230" rpy="0 0 0" />
+          <inertia ixx="0.00041540"  ixy="0.00000000" ixz="0.00000010"
+                                   iyy="0.00041637" iyz="-0.00004589"
+                                                    izz="0.00002982"/>
+        </inertial>
+      </xacro:unless>
+      <xacro:if value="${is_right}">
+        <!-- Right upper leg inertia -->
+        <inertial>
+          <mass value="0.14737324"/>
+          <origin xyz="-0.00001530 -0.01767640 -0.07838230" rpy="0 0 0" />
+          <inertia ixx="0.00041540"  ixy="0.00000000" ixz="-0.00000010"
+                                   iyy="0.00041637" iyz="0.00004589"
+                                                    izz="0.00002982"/>
+        </inertial>
+      </xacro:if>
+      <!-- UPPER LEG LINK VISUAL -->
+      <visual>
+        <origin xyz="0 0 0" rpy="0 0 0" />
+        <geometry>
+          <xacro:unless value="${is_right}">
+            <mesh filename="file://$(find ros2_description_bolt)/meshes/${mesh_ext}/without_foot/solo_upper_leg_left_side.${mesh_ext}"/>
+            <!-- <mesh filename="package://robot_properties_solo/resources/meshes/${mesh_ext}/without_foot/solo_upper_leg_left_side.${mesh_ext}"/> -->
+          </xacro:unless>
+          <xacro:if value="${is_right}">
+            <mesh filename="file://$(find ros2_description_bolt)/meshes/${mesh_ext}/without_foot/solo_upper_leg_right_side.${mesh_ext}"/>
+            <!-- <mesh filename="package://robot_properties_solo/resources/meshes/${mesh_ext}/without_foot/solo_upper_leg_right_side.${mesh_ext}"/> -->
+          </xacro:if>
+        </geometry>
+        <material name="${color_name}">
+            <color rgba="${color} ${opacity}"/>
+        </material>
+      </visual>
+      <!-- UPPER LEG LINK COLLISION -->
+      <collision>
+        <origin xyz="0 0 0" rpy="0 0 0" />
+        <geometry>
+          <xacro:unless value="${is_right}">
+            <mesh filename="file://$(find ros2_description_bolt)/meshes/${mesh_ext}/without_foot/solo_upper_leg_left_side.${mesh_ext}"/>
+            <!-- <mesh filename="package://robot_properties_solo/resources/meshes/${mesh_ext}/without_foot/solo_upper_leg_left_side.${mesh_ext}"/> -->
+          </xacro:unless>
+          <xacro:if value="${is_right}">
+            <mesh filename="file://$(find ros2_description_bolt)/meshes/${mesh_ext}/without_foot/solo_upper_leg_right_side.${mesh_ext}"/>
+            <!-- <mesh filename="package://robot_properties_solo/resources/meshes/${mesh_ext}/without_foot/solo_upper_leg_right_side.${mesh_ext}"/> -->
+          </xacro:if>
+        </geometry>
+        <material name="${color_name}">
+            <color rgba="${color} ${opacity}"/>
+        </material>
+      </collision>
+      <!-- Bullet specific paramters -->
+      <!-- <contact>
+        <lateral_friction value="1.0"/>
+        <restitution value="0.5"/>
+      </contact> -->
+    </link> <!-- END UPPER LEG LINK -->
+  <!-- KFE JOINT-->
+    <joint name="${prefix}_KFE" type="revolute">
+      <parent link="${prefix}_UPPER_LEG"/>
+      <child link="${prefix}_LOWER_LEG"/>
+      <limit lower="-3.14" upper="3.14" velocity="1" effort="7"/>
+      <!-- <limit effort="1000" lower="-10" upper="10" velocity="1000"/> -->
+      <!-- joints rotates around the y-axis -->
+      <axis xyz="0 1 0"/>
+      <!-- placement of the joint -->
+      <xacro:if value="${is_front}">
+        <xacro:unless value="${is_right}">
+          <origin xyz="0 ${HFE_2_KFE_y} ${-HFE_2_KFE_z}" rpy="0 0 0" />
+        </xacro:unless>
+        <xacro:if value="${is_right}">
+          <origin xyz="0 ${-HFE_2_KFE_y} ${-HFE_2_KFE_z}" rpy="0 0 0" />
+        </xacro:if>
+      </xacro:if>
+      <xacro:unless value="${is_front}">
+        <xacro:unless value="${is_right}">
+          <origin xyz="0 ${HFE_2_KFE_y} ${-HFE_2_KFE_z}" rpy="0 0 0" />
+        </xacro:unless>
+        <xacro:if value="${is_right}">
+          <origin xyz="0 ${-HFE_2_KFE_y} ${-HFE_2_KFE_z}" rpy="0 0 0" />
+        </xacro:if>
+      </xacro:unless>
+      <!-- pybullet simulation parameters -->
+      <dynamics damping="1.0" friction="1000.0"/>
+    </joint>
+  <!-- LOWER LEG LINK -->
+    <link name="${prefix}_LOWER_LEG">
+      <!-- LOWER LEG LINK INERTIAL -->
+      <xacro:unless value="${is_right}">
+        <!-- Left lower leg inertia -->
+        <inertial>
+          <mass value="0.02318294"/>
+          <origin xyz="0.00000000 0.00776716 -0.07003876" rpy="0 0 0" />
+          <inertia ixx="0.00008508" ixy="0.00000000"  ixz="0.00000000"
+                                  iyy="0.00008580"  iyz="-0.00000200"
+                                                    izz="0.00000139"/>
+        </inertial>
+      </xacro:unless>
+      <xacro:if value="${is_right}">
+        <!-- Right lower leg inertia -->
+        <inertial>
+          <mass value="0.02318294"/>
+          <origin xyz="0.00000000 -0.00776716 -0.07003876" rpy="0 0 0" />
+          <inertia ixx="0.00008508" ixy="0.00000000"  ixz="0.00000000"
+                                  iyy="0.00008580"  iyz="0.00000200"
+                                                    izz="0.00000139"/>
+        </inertial>
+      </xacro:if>
+      <!-- LOWER LEG LINK VISUAL -->
+      <visual>
+        <origin xyz="0 0 0" rpy="0 0 0" />
+        <geometry>
+          <xacro:unless value="${is_right}">
+            <mesh filename="file://$(find ros2_description_bolt)/meshes/${mesh_ext}/without_foot/solo_lower_leg_v2_left_side.${mesh_ext}"/>
+            <!-- <mesh filename="package://robot_properties_solo/resources/meshes/${mesh_ext}/without_foot/solo_lower_leg_v2_left_side.${mesh_ext}"/> -->
+          </xacro:unless>
+          <xacro:if value="${is_right}">
+            <mesh filename="file://$(find ros2_description_bolt)/meshes/${mesh_ext}/without_foot/solo_lower_leg_v2_right_side.${mesh_ext}"/>
+            <!-- <mesh filename="package://robot_properties_solo/resources/meshes/${mesh_ext}/without_foot/solo_lower_leg_v2_right_side.${mesh_ext}"/> -->
+          </xacro:if>
+        </geometry>
+        <material name="${color_name}">
+            <color rgba="${color} ${opacity}"/>
+        </material>
+      </visual>
+      <!-- LOWER LEG LINK COLLISION -->
+      <collision>
+        <origin xyz="0 0 0" rpy="0 0 0" />
+        <geometry>
+          <xacro:unless value="${is_right}">
+            <mesh filename="file://$(find ros2_description_bolt)/meshes/${mesh_ext}/without_foot/solo_lower_leg_v2_left_side.${mesh_ext}"/>
+            <!-- <mesh filename="package://robot_properties_solo/resources/meshes/${mesh_ext}/without_foot/solo_lower_leg_v2_left_side.${mesh_ext}"/> -->
+          </xacro:unless>
+          <xacro:if value="${is_right}">
+            <mesh filename="file://$(find ros2_description_bolt)/meshes/${mesh_ext}/without_foot/solo_lower_leg_v2_right_side.${mesh_ext}"/>
+            <!-- <mesh filename="package://robot_properties_solo/resources/meshes/${mesh_ext}/without_foot/solo_lower_leg_v2_right_side.${mesh_ext}"/> -->
+          </xacro:if>
+        </geometry>
+        <material name="${color_name}">
+            <color rgba="${color} ${opacity}"/>
+        </material>
+      </collision>
+      <!-- Bullet specific paramters -->
+      <!-- <contact>
+        <lateral_friction value="1.0"/>
+        <restitution value="0.5"/>
+      </contact> -->
+        <contact>
+            <min_depth>0.001</min_depth>
+        </contact>
+        <mu1>200.0</mu1>
+        <mu2>100.0</mu2>
+        <kp>1e13</kp>
+        <kd>1.0</kd>
+        <minDepth>0.001</minDepth>
+        <bounce_threshold>10000000</bounce_threshold>
+        <maxVel>0.1</maxVel>
+        <fdir1>0 0 0</fdir1>
+    </link> <!-- END LOWER LEG LINK -->
+     <!-- NO SIDE MOTION-->
     <xacro:unless value="${has_side_motion}">
       <!-- Joint between the base and the ${prefix} upper leg -->
@@ -212,198 +385,4 @@
       </joint>
     </xacro:unless>
-    <link name="${prefix}_UPPER_LEG">
-      <!-- UPPER LEG LINK INERTIAL -->
-      <xacro:unless value="${is_right}">
-        <!-- Left upper leg inertia -->
-        <inertial>
-        <!-- <origin rpy="0 0 0" xyz="0.00001377 0.01935853 -0.07870700"/> -->
-        <!-- <mass value="0.14853845"/> -->
-        <!-- <inertia ixx="0.00041107" ixy="0.0" ixz="0.0" iyy="0.00041193" iyz="0.00004671" izz="0.00003024"/> -->
-        <mass value="0.14737324"/>
-        <origin xyz="0.00001530 0.01767640 -0.07838230" rpy="0 0 0" />
-        <inertia ixx="0.00041540"  ixy="0.00000000" ixz="0.00000010"
-                                   iyy="0.00041637" iyz="-0.00004589"
-                                                    izz="0.00002982"/>
-        </inertial>
-      </xacro:unless>
-      <xacro:if value="${is_right}">
-        <!-- Right upper leg inertia -->
-        <inertial>
-        <!-- <origin rpy="0 0 0" xyz="0.00001377 0.01935853 -0.07870700"/> -->
-        <!-- <mass value="0.14853845"/> -->
-        <!-- <inertia ixx="0.00041107" ixy="0.0" ixz="0.0" iyy="0.00041193" iyz="0.00004671" izz="0.00003024"/> -->
-        <mass value="0.14737324"/>
-        <origin xyz="-0.00001530 -0.01767640 -0.07838230" rpy="0 0 0" />
-        <inertia ixx="0.00041540"  ixy="0.00000000" ixz="-0.00000010"
-                                   iyy="0.00041637" iyz="0.00004589"
-                                                    izz="0.00002982"/>
-        </inertial>
-      </xacro:if>
-      <!-- UPPER LEG LINK VISUAL -->
-      <visual>
-        <origin xyz="0 0 0" rpy="0 0 0" />
-        <geometry>
-          <xacro:unless value="${is_right}">
-            <mesh filename="file://$(find ros2_description_bolt)/meshes/${mesh_ext}/without_foot/solo_upper_leg_left_side.${mesh_ext}"/>
-            <!-- <mesh filename="package://robot_properties_solo/resources/meshes/${mesh_ext}/without_foot/solo_upper_leg_left_side.${mesh_ext}"/> -->
-          </xacro:unless>
-          <xacro:if value="${is_right}">
-            <mesh filename="file://$(find ros2_description_bolt)/meshes/${mesh_ext}/without_foot/solo_upper_leg_right_side.${mesh_ext}"/>
-            <!-- <mesh filename="package://robot_properties_solo/resources/meshes/${mesh_ext}/without_foot/solo_upper_leg_right_side.${mesh_ext}"/> -->
-          </xacro:if>
-        </geometry>
-        <material name="${color_name}">
-            <color rgba="${color} ${opacity}"/>
-        </material>
-      </visual>
-      <!-- UPPER LEG LINK COLLISION -->
-      <collision>
-        <origin xyz="0 0 0" rpy="0 0 0" />
-        <geometry>
-          <xacro:unless value="${is_right}">
-            <mesh filename="file://$(find ros2_description_bolt)/meshes/${mesh_ext}/without_foot/solo_upper_leg_left_side.${mesh_ext}"/>
-            <!-- <mesh filename="package://robot_properties_solo/resources/meshes/${mesh_ext}/without_foot/solo_upper_leg_left_side.${mesh_ext}"/> -->
-          </xacro:unless>
-          <xacro:if value="${is_right}">
-            <mesh filename="file://$(find ros2_description_bolt)/meshes/${mesh_ext}/without_foot/solo_upper_leg_right_side.${mesh_ext}"/>
-            <!-- <mesh filename="package://robot_properties_solo/resources/meshes/${mesh_ext}/without_foot/solo_upper_leg_right_side.${mesh_ext}"/> -->
-          </xacro:if>
-        </geometry>
-        <material name="${color_name}">
-            <color rgba="${color} ${opacity}"/>
-        </material>
-      </collision>
-      <!-- Bullet specific paramters -->
-      <contact>
-        <lateral_friction value="1.0"/>
-        <restitution value="0.5"/>
-      </contact>
-    </link> <!-- END UPPER LEG LINK -->
-    <!-- KFE: Joint between the upper leg and the lower leg -->
-    <joint name="${prefix}_KFE" type="revolute">
-      <parent link="${prefix}_UPPER_LEG"/>
-      <child link="${prefix}_LOWER_LEG"/>
-      <limit effort="1000" lower="-10" upper="10" velocity="1000"/>
-      <!-- joints rotates around the y-axis -->
-      <axis xyz="0 1 0"/>
-      <!-- placement of the joint -->
-      <xacro:if value="${is_front}">
-        <xacro:unless value="${is_right}">
-          <origin xyz="0 ${HFE_2_KFE_y} ${-HFE_2_KFE_z}" rpy="0 0 0" />
-        </xacro:unless>
-        <xacro:if value="${is_right}">
-          <origin xyz="0 ${-HFE_2_KFE_y} ${-HFE_2_KFE_z}" rpy="0 0 0" />
-        </xacro:if>
-      </xacro:if>
-      <xacro:unless value="${is_front}">
-        <xacro:unless value="${is_right}">
-          <origin xyz="0 ${HFE_2_KFE_y} ${-HFE_2_KFE_z}" rpy="0 0 0" />
-        </xacro:unless>
-        <xacro:if value="${is_right}">
-          <origin xyz="0 ${-HFE_2_KFE_y} ${-HFE_2_KFE_z}" rpy="0 0 0" />
-        </xacro:if>
-      </xacro:unless>
-      <!-- pybullet simulation parameters -->
-      <dynamics damping="0.0" friction="0.0"/>
-    </joint>
-    <link name="${prefix}_LOWER_LEG">
-      <!-- LOWER LEG LINK INERTIAL -->
-      <xacro:unless value="${is_right}">
-        <!-- Left lower leg inertia -->
-        <inertial>
-        <!-- <origin rpy="0 0 0" xyz="0.0 0.00787644 -0.08928215"/> -->
-        <!-- <mass value="0.03070001"/> -->
-        <!-- <inertia ixx="0.00012024" ixy="0.0" ixz="0.0" iyy="0.00012029" iyz="0.00000305" izz="0.00000216"/> -->
-        <mass value="0.02318294"/>
-        <origin xyz="0.00000000 0.00776716 -0.07003876" rpy="0 0 0" />
-        <inertia ixx="0.00008508" ixy="0.00000000"  ixz="0.00000000"
-                                  iyy="0.00008580"  iyz="-0.00000200"
-                                                    izz="0.00000139"/>
-        </inertial>
-      </xacro:unless>
-      <xacro:if value="${is_right}">
-        <!-- Right lower leg inertia -->
-        <inertial>
-        <!-- <origin rpy="0 0 0" xyz="0.0 0.00787644 -0.08928215"/> -->
-        <!-- <mass value="0.03070001"/> -->
-        <!-- <inertia ixx="0.00012024" ixy="0.0" ixz="0.0" iyy="0.00012029" iyz="0.00000305" izz="0.00000216"/> -->
-        <mass value="0.02318294"/>
-        <origin xyz="0.00000000 -0.00776716 -0.07003876" rpy="0 0 0" />
-        <inertia ixx="0.00008508" ixy="0.00000000"  ixz="0.00000000"
-                                  iyy="0.00008580"  iyz="0.00000200"
-                                                    izz="0.00000139"/>
-        </inertial>
-      </xacro:if>
-      <!-- LOWER LEG LINK VISUAL -->
-      <visual>
-        <origin xyz="0 0 0" rpy="0 0 0" />
-        <geometry>
-          <xacro:unless value="${is_right}">
-            <mesh filename="file://$(find ros2_description_bolt)/meshes/${mesh_ext}/without_foot/solo_lower_leg_v2_left_side.${mesh_ext}"/>
-            <!-- <mesh filename="package://robot_properties_solo/resources/meshes/${mesh_ext}/without_foot/solo_lower_leg_v2_left_side.${mesh_ext}"/> -->
-          </xacro:unless>
-          <xacro:if value="${is_right}">
-            <mesh filename="file://$(find ros2_description_bolt)/meshes/${mesh_ext}/without_foot/solo_lower_leg_v2_right_side.${mesh_ext}"/>
-            <!-- <mesh filename="package://robot_properties_solo/resources/meshes/${mesh_ext}/without_foot/solo_lower_leg_v2_right_side.${mesh_ext}"/> -->
-          </xacro:if>
-        </geometry>
-        <material name="${color_name}">
-            <color rgba="${color} ${opacity}"/>
-        </material>
-      </visual>
-      <!-- LOWER LEG LINK COLLISION -->
-      <collision>
-        <origin xyz="0 0 0" rpy="0 0 0" />
-        <geometry>
-          <xacro:unless value="${is_right}">
-            <mesh filename="file://$(find ros2_description_bolt)/meshes/${mesh_ext}/without_foot/solo_lower_leg_v2_left_side.${mesh_ext}"/>
-            <!-- <mesh filename="package://robot_properties_solo/resources/meshes/${mesh_ext}/without_foot/solo_lower_leg_v2_left_side.${mesh_ext}"/> -->
-          </xacro:unless>
-          <xacro:if value="${is_right}">
-            <mesh filename="file://$(find ros2_description_bolt)/meshes/${mesh_ext}/without_foot/solo_lower_leg_v2_right_side.${mesh_ext}"/>
-            <!-- <mesh filename="package://robot_properties_solo/resources/meshes/${mesh_ext}/without_foot/solo_lower_leg_v2_right_side.${mesh_ext}"/> -->
-          </xacro:if>
-        </geometry>
-        <material name="${color_name}">
-            <color rgba="${color} ${opacity}"/>
-        </material>
-      </collision>
-      <!-- Bullet specific paramters -->
-      <contact>
-        <lateral_friction value="1.0"/>
-        <restitution value="0.5"/>
-      </contact>
-    </link> <!-- END LOWER LEG LINK -->
-    <!-- Joint between the lower leg and the ankle,
-         this is only a dummy joint such that we
-         can assign coordinate frames to foot-->
-    <joint name="${prefix}_ANKLE" type="fixed">
-      <parent link="${prefix}_LOWER_LEG"/>
-      <child link="${prefix}_FOOT"/>
-      <!-- Joint placement -->
-      <xacro:unless value="${is_right}">
-        <origin xyz="0 ${KFE_2_FOOT_y} ${-KFE_2_FOOT_z}" rpy="0 0 0" />
-      </xacro:unless>
-      <xacro:if value="${is_right}">
-        <origin xyz="0 ${-KFE_2_FOOT_y} ${-KFE_2_FOOT_z}" rpy="0 0 0" />
-      </xacro:if>
-      <!-- Limits -->
-      <limit effort="1000" lower="-10" upper="10" velocity="1000"/>
-      <!-- pybullet simulation parameters -->
-      <dynamics damping="0.0" friction="0.0"/>
-    </joint>
-    <link name="${prefix}_FOOT">
-      <!-- FOOT INERTIAL -->
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
File: ros2_control_solo/ros2_description_bolt/urdf/solo_xacro/solo12.urdf.xacro (robot description, xacro)
@@ -21,7 +21,4 @@
                                                       izz="0.01605370"
           />
-          <!-- <mass value="1.16115091"/> -->
-          <!-- The base is extremely symmetrical. -->
-          <!-- <inertia ixx="0.00578574" ixy="0.0" ixz="0.0" iyy="0.01938108" iyz="0.0" izz="0.02476124"/> -->
       </inertial>
       <!-- BASE LINK VISUAL -->
@@ -48,8 +45,8 @@
       </collision>
       <!-- Bullet specific paramters -->
-      <contact>
+      <!-- <contact>
         <lateral_friction value="1.0"/>
         <restitution value="0.5"/>
-      </contact>
+      </contact> -->
     </link> <!-- END BASE LINK -->
     <!-- Include the legs -->
