Commit message: no more slipping

File: ros2_control_solo/ros2_description_bolt/ros2_control/system_solo.ros2_control.xacro (robot description, xacro)
@@ -14,5 +14,7 @@
           <param name="max">3.14</param>
         </command_interface>
-       <state_interface name="position"/>
+       <state_interface name="position">
+          <!-- <param name="initial_value">0.0001</param> -->
+        </state_interface>
         <state_interface name="velocity"/>
         <state_interface name="effort"/>
@@ -23,5 +25,7 @@
           <param name="max">3.14</param>
         </command_interface>
-        <state_interface name="position"/>
+        <state_interface name="position">
+          <!-- <param name="initial_value">0.0001</param> -->
+        </state_interface>
         <state_interface name="velocity"/>
         <state_interface name="effort"/>
@@ -32,5 +36,7 @@
           <param name="max">3.14</param>
         </command_interface>
-       <state_interface name="position"/>
+       <state_interface name="position">
+          <!-- <param name="initial_value">0.0001</param> -->
+        </state_interface>
         <state_interface name="velocity"/>
         <state_interface name="effort"/>
@@ -41,5 +47,7 @@
           <param name="max">3.14</param>
         </command_interface>
-       <state_interface name="position"/>
+       <state_interface name="position">
+          <!-- <param name="initial_value">0.0001</param> -->
+        </state_interface>
         <state_interface name="velocity"/>
         <state_interface name="effort"/>

File: ros2_control_solo/ros2_description_bolt/urdf/solo_xacro/leg.xacro (robot description, xacro)
@@ -44,5 +44,5 @@
         </xacro:unless>
         <!-- pybullet simulation parameters -->
-        <dynamics friction="10.0"/>
+        <dynamics damping="0.7" friction="1.0"/>
         <!-- <dynamics damping="0.0" friction="0.0"/> -->
       </joint>
@@ -128,5 +128,5 @@
           <xacro:if value="${is_front}">
             <xacro:unless value="${is_right}">
-              <!-- HAA body inertia -->
+              <!-- Hip FE FL inertia -->
               <origin xyz="-0.09407251 -0.00438935 0.00001384" rpy="0 0 0" />
               <inertia ixx="0.00002802" ixy="0.00003687" ixz="-0.00000009"
@@ -135,5 +135,5 @@
             </xacro:unless>
             <xacro:if value="${is_right}">
-              <!-- HAA body inertia -->
+              <!-- Hip FE FR inertia -->
               <origin xyz="-0.09407251 0.00438935 -0.00001384" rpy="0 0 0" />
               <inertia ixx="0.00002802" ixy="-0.00003687" ixz="0.00000009"
@@ -144,5 +144,5 @@
           <xacro:unless value="${is_front}">
             <xacro:unless value="${is_right}">
-              <!-- HAA body inertia -->
+              <!-- Hip FE HL inertia -->
               <origin xyz="0.09407251 -0.00438935 -0.00001384" rpy="0 0 0" />
               <inertia ixx="0.00002802" ixy="-0.00003687" ixz="-0.00000009"
@@ -151,5 +151,5 @@
             </xacro:unless>
             <xacro:if value="${is_right}">
-              <!-- HAA body inertia -->
+              <!-- Hip FE HR inertia -->
               <origin xyz="0.09407251 0.00438935 0.00001384" rpy="0 0 0" />
               <inertia ixx="0.00002802" ixy="0.00003687" ixz="0.00000009"
@@ -187,5 +187,5 @@
         <!-- pybullet simulation parameters -->
         <!-- <dynamics damping="0.0" friction="0.0"/> -->
-        <dynamics friction="10.0"/>
+        <dynamics damping="0.7" friction="1.0"/>
       </joint>
     </xacro:if>
@@ -248,8 +248,8 @@
       </collision>
       <!-- Bullet specific paramters -->
-      <!-- <contact>
+      <contact>
         <lateral_friction value="1.0"/>
         <restitution value="0.5"/>
-      </contact> -->
+      </contact>
     </link> <!-- END UPPER LEG LINK -->
   <!-- KFE JOINT-->
@@ -279,5 +279,6 @@
       </xacro:unless>
       <!-- pybullet simulation parameters -->
-      <dynamics damping="1.0" friction="1000.0"/>
+      <!-- <dynamics damping="1.0" friction="1000.0"/> -->
+      <dynamics damping="0.7" friction="1.0"/>
     </joint>
   <!-- LOWER LEG LINK -->
@@ -339,20 +340,54 @@
       </collision>
       <!-- Bullet specific paramters -->
-      <!-- <contact>
+      <contact>
         <lateral_friction value="1.0"/>
         <restitution value="0.5"/>
-      </contact> -->
-        <contact>
+      </contact>
+        <!-- <contact>
             <min_depth>0.001</min_depth>
         </contact>
         <mu1>200.0</mu1>
         <mu2>100.0</mu2>
-        <kp>1e13</kp>
+        <kp>1000000.0</kp>
         <kd>1.0</kd>
         <minDepth>0.001</minDepth>
         <bounce_threshold>10000000</bounce_threshold>
-        <maxVel>0.1</maxVel>
-        <fdir1>0 0 0</fdir1>
+        <maxVel>0.0</maxVel>
+        <fdir1>0 0 0</fdir1> -->
+        <kp>1000000.0</kp>
+        <kd>1.0</kd>
+        <mu1>0.8</mu1>
+        <mu2>0.8</mu2>
+        <maxVel>0.0</maxVel>
+        <minDepth>0.001</minDepth>
     </link> <!-- END LOWER LEG LINK -->
+    <!-- Joint between the lower leg and the ankle,
+      this is only a dummy joint such that we
+      can assign coordinate frames to foot-->
+    <joint name="${prefix}_ANKLE" type="fixed">
+      <parent link="${prefix}_LOWER_LEG"/>
+      <child link="${prefix}_FOOT"/>
+      <!-- Joint placement -->
+      <xacro:unless value="${is_right}">
+        <origin xyz="0 ${KFE_2_FOOT_y} ${-KFE_2_FOOT_z}" rpy="0 0 0" />
+      </xacro:unless>
+      <xacro:if value="${is_right}">
+        <origin xyz="0 ${-KFE_2_FOOT_y} ${-KFE_2_FOOT_z}" rpy="0 0 0" />
+      </xacro:if>
+      <!-- Limits -->
+      <limit effort="1000" lower="-10" upper="10" velocity="1000"/>
+      <!-- pybullet simulation parameters -->
+      <dynamics damping="0.7" friction="1.0"/>
+    </joint>
+    <link name="${prefix}_FOOT">
+      <!-- FOOT INERTIAL -->
+      <inertial>
+        <origin xyz="0 0 0" rpy="0 0 0" />
+        <mass value="0.0"/>
+        <inertia ixx="0.0" ixy="0.0" ixz="0.0"
+                           iyy="0.0" iyz="0.0"
+                                     izz="0.0"/>
+      </inertial>
+    </link> <!-- END FOOT LINK -->
      <!-- NO SIDE MOTION-->
     <xacro:unless value="${has_side_motion}">
@@ -361,5 +396,5 @@
         <parent link="base_link"/>
         <child link="${prefix}_UPPER_LEG"/>
-        <limit effort="1000" lower="-10" upper="10" velocity="1000"/>
+        <limit lower="-3.14" upper="3.14" velocity="1" effort="7"/>
         <!-- joints rotates around the y-axis -->
         <axis xyz="0 1 0"/>
@@ -382,5 +417,5 @@
         </xacro:unless>
         <!-- pybullet simulation parameters -->
-        <dynamics damping="0.0" friction="0.0"/>
+        <dynamics damping="1.0" friction="1000.0"/>
       </joint>
     </xacro:unless>
